File: Examples/RLC/RLC.sch (KiCad schematic (older format))
At the start: 6 parts, among them U1 plot_v1, U2 plot_v1

Commit message: Added new subckts
Parts:
- L1: symbol L -> L-RESCUE-RLC
- R1: symbol R -> R-RESCUE-RLC
Changed lines of the file:
@@
 EESchema Schematic File Version 2
+LIBS:RLC-rescue
 LIBS:eSim_Analog
 LIBS:eSim_Devices
@@
 $EndDescr
 $Comp
-L R R1
+L R-RESCUE-RLC R1
 U 1 1 56C172A1
 P 4850 2700
@@
 $EndComp
 $Comp
-L L L1
+L L-RESCUE-RLC L1
 U 1 1 56C172D6
 P 3800 3200
