File: Examples/74LS283-test/74LS283-test.sch (KiCad schematic (older format))
At the start: 21 parts, among them U1 plot_v1, U2 plot_v1, U3 plot_v1, U4 plot_v1, U5 plot_v1, X1 eSim_74LS283

Commit message: Supporting examples added
Parts:
- removed v4, v5, v7, v8: 5, R1, symbol DC
- added v4, v5, v7, v8: pulse, R1, symbol pulse
- v10, v3: value 0 -> 5
- v9: value 5 -> 0
Connections:
- net GND: now also v4.2 (-), v5.2 (-), v7.2 (-), v8.2 (-)
- net at X1.12 (A4): now also v8.1 (+)
- net at X1.14 (A3): now also v7.1 (+)
- net at X1.3 (A2): now also v4.1 (+)
- net at X1.6 (A1): now also v5.1 (+)
Changed lines of the file:
@@
-$EndComp
-$Comp
-L DC v5
-U 1 1 5E2027C8
-P 3850 3500
-F 0 "v5" H 3650 3600 60  0000 C CNN
-F 1 "5" H 3650 3450 60  0000 C CNN
-F 2 "R1" H 3550 3500 60  0000 C CNN
-F 3 "" H 3850 3500 60  0000 C CNN
-	1    3850 3500
-	0    1    1    0
-$EndComp
-$Comp
-L DC v4
-U 1 1 5E202908
-P 3850 3050
-F 0 "v4" H 3650 3150 60  0000 C CNN
-F 1 "5" H 3650 3000 60  0000 C CNN
-F 2 "R1" H 3550 3050 60  0000 C CNN
-F 3 "" H 3850 3050 60  0000 C CNN
-	1    3850 3050
-	0    1    1    0
-$EndComp
-$Comp
-L DC v8
-U 1 1 5E20295C
-P 8450 3350
-F 0 "v8" H 8250 3450 60  0000 C CNN
-F 1 "5" H 8250 3300 60  0000 C CNN
-F 2 "R1" H 8150 3350 60  0000 C CNN
-F 3 "" H 8450 3350 60  0000 C CNN
-	1    8450 3350
-	0    -1   -1   0
-$EndComp
-$Comp
-L DC v7
-U 1 1 5E202A5C
-P 8450 3050
-F 0 "v7" H 8250 3150 60  0000 C CNN
-F 1 "5" H 8250 3000 60  0000 C CNN
-F 2 "R1" H 8150 3050 60  0000 C CNN
-F 3 "" H 8450 3050 60  0000 C CNN
-	1    8450 3050
-	0    -1   -1   0
 $EndComp
 $Comp
@@
 P 9100 3500
 F 0 "v10" H 8900 3600 60  0000 C CNN
-F 1 "0" H 8900 3450 60  0000 C CNN
+F 1 "5" H 8900 3450 60  0000 C CNN
 F 2 "R1" H 8800 3500 60  0000 C CNN
 F 3 "" H 9100 3500 60  0000 C CNN
@@
 P 9100 2900
 F 0 "v9" H 8900 3000 60  0000 C CNN
-F 1 "5" H 8900 2850 60  0000 C CNN
+F 1 "0" H 8900 2850 60  0000 C CNN
 F 2 "R1" H 8800 2900 60  0000 C CNN
 F 3 "" H 9100 2900 60  0000 C CNN
@@
 P 3200 3650
 F 0 "v3" H 3000 3750 60  0000 C CNN
-F 1 "0" H 3000 3600 60  0000 C CNN
+F 1 "5" H 3000 3600 60  0000 C CNN
 F 2 "R1" H 2900 3650 60  0000 C CNN
 F 3 "" H 3200 3650 60  0000 C CNN
@@
 	1    0    0    -1
 $EndComp
+$Comp
+L pulse v4
+U 1 1 5E283423
+P 3850 3050
+F 0 "v4" H 3650 3150 60  0000 C CNN
+F 1 "pulse" H 3650 3000 60  0000 C CNN
+F 2 "R1" H 3550 3050 60  0000 C CNN
+F 3 "" H 3850 3050 60  0000 C CNN
+	1    3850 3050
+	0    1    1    0
+$EndComp
+$Comp
+L pulse v5
+U 1 1 5E283495
+P 3850 3500
+F 0 "v5" H 3650 3600 60  0000 C CNN
+F 1 "pulse" H 3650 3450 60  0000 C CNN
+F 2 "R1" H 3550 3500 60  0000 C CNN
+F 3 "" H 3850 3500 60  0000 C CNN
+	1    3850 3500
+	0    1    1    0
+$EndComp
+$Comp
+L pulse v7
+U 1 1 5E283A52
+P 8450 3050
+F 0 "v7" H 8250 3150 60  0000 C CNN
+F 1 "pulse" H 8250 3000 60  0000 C CNN
+F 2 "R1" H 8150 3050 60  0000 C CNN
+F 3 "" H 8450 3050 60  0000 C CNN
+	1    8450 3050
+	0    -1   1    0
+$EndComp
+$Comp
+L pulse v8
+U 1 1 5E283B03
+P 8450 3350
+F 0 "v8" H 8250 3450 60  0000 C CNN
+F 1 "pulse" H 8250 3300 60  0000 C CNN
+F 2 "R1" H 8150 3350 60  0000 C CNN
+F 3 "" H 8450 3350 60  0000 C CNN
+	1    8450 3350
+	0    -1   -1   0
+$EndComp
 $EndSCHEMATC
