File: Examples/74LS283-test/74LS283.sch (KiCad schematic (older format))
At the start: 28 parts, among them Q1 eSim_NPN, Q2 eSim_NPN, Q3 eSim_NPN, Q4 eSim_NPN, Q5 eSim_NPN, U1 PORT, U2 d_inverter, U3 d_inverter, U4 d_inverter, U5 dac_bridge_5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

Commit message: Supporting examples added
Parts:
- added R11, R12, R13, R14, R15: 100k, symbol eSim_R
Connections:
- net at Q5.1 (C), R10.2, U1.4: now also R15.1
- net at Q1.3 (E), Q2.3 (E), Q3.3 (E)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: now also R11.2, R12.2, R13.2, R14.2, R15.2
- net at Q4.1 (C), R8.2, U1.1: now also R14.1
- net at Q3.1 (C), R6.2, U1.13: now also R13.1
- net at Q2.1 (C), R4.2, U1.10: now also R12.1
- net at Q1.1 (C), R2.2, U1.9: now also R11.1
