File: Examples/74LS83A-test/74LS83A-test.sch (KiCad schematic (older format))
At the start: 22 parts, among them U1 plot_v1, U2 plot_v1, U3 plot_v1, U4 plot_v1, U5 plot_v1, U6 plot_v1, X1 eSim_74LS83A

Commit message: Supporting examples added
Parts:
- removed v3, v4, v5, v6: 5, R1, symbol DC
- added v3, v4, v5, v6: pulse, R1, symbol pulse
- v9: value 0 -> 5
Connections:
- net GND: now also v3.2 (-), v4.2 (-), v5.2 (-), v6.2 (-)
- net at X1.1 (A4): now also v4.1 (+)
- net at X1.10 (A1): now also v6.1 (+)
- net at X1.3 (A3): now also v3.1 (+)
- net at X1.8 (A2): now also v5.1 (+)
Other:
- note added: "A3"
- note added: "A4"
- note added: "a1\n"
- note added: "a2"
- note added: "carry_in\n"
Changed lines of the file:
@@
-$EndComp
-$Comp
-L DC v3
-U 1 1 5E1F2EBA
-P 4250 2400
-F 0 "v3" H 4050 2500 60  0000 C CNN
-F 1 "5" H 4050 2350 60  0000 C CNN
-F 2 "R1" H 3950 2400 60  0000 C CNN
-F 3 "" H 4250 2400 60  0000 C CNN
-	1    4250 2400
-	0    1    1    0
-$EndComp
-$Comp
-L DC v4
-U 1 1 5E1F2F73
-P 4250 2950
-F 0 "v4" H 4050 3050 60  0000 C CNN
-F 1 "5" H 4050 2900 60  0000 C CNN
-F 2 "R1" H 3950 2950 60  0000 C CNN
-F 3 "" H 4250 2950 60  0000 C CNN
-	1    4250 2950
-	0    1    1    0
 $EndComp
 $Comp
@@
 	0    -1   1    0
 $EndComp
-$Comp
-L DC v6
-U 1 1 5E1F336F
-P 7800 3800
-F 0 "v6" H 7600 3900 60  0000 C CNN
-F 1 "5" H 7600 3750 60  0000 C CNN
-F 2 "R1" H 7500 3800 60  0000 C CNN
-F 3 "" H 7800 3800 60  0000 C CNN
-	1    7800 3800
-	0    -1   1    0
-$EndComp
-$Comp
-L DC v5
-U 1 1 5E1F3375
-P 4800 3950
-F 0 "v5" H 4600 4050 60  0000 C CNN
-F 1 "5" H 4600 3900 60  0000 C CNN
-F 2 "R1" H 4500 3950 60  0000 C CNN
-F 3 "" H 4800 3950 60  0000 C CNN
-	1    4800 3950
-	0    1    -1   0
-$EndComp
 Wire Wire Line
 	7350 3800 6650 3800
@@
 P 8800 3550
 F 0 "v9" H 8600 3650 60  0000 C CNN
-F 1 "0" H 8600 3500 60  0000 C CNN
+F 1 "5" H 8600 3500 60  0000 C CNN
 F 2 "R1" H 8500 3550 60  0000 C CNN
 F 3 "" H 8800 3550 60  0000 C CNN
@@
 	0    1    1    0
 $EndComp
+$Comp
+L pulse v3
+U 1 1 5E282F1D
+P 4250 2400
+F 0 "v3" H 4050 2500 60  0000 C CNN
+F 1 "pulse" H 4050 2350 60  0000 C CNN
+F 2 "R1" H 3950 2400 60  0000 C CNN
+F 3 "" H 4250 2400 60  0000 C CNN
+	1    4250 2400
+	0    1    1    0
+$EndComp
+$Comp
+L pulse v4
+U 1 1 5E282F90
+P 4250 2950
+F 0 "v4" H 4050 3050 60  0000 C CNN
+F 1 "pulse" H 4050 2900 60  0000 C CNN
+F 2 "R1" H 3950 2950 60  0000 C CNN
+F 3 "" H 4250 2950 60  0000 C CNN
+	1    4250 2950
+	0    1    1    0
+$EndComp
+$Comp
+L pulse v5
+U 1 1 5E282FE9
+P 4800 3950
+F 0 "v5" H 4600 4050 60  0000 C CNN
+F 1 "pulse" H 4600 3900 60  0000 C CNN
+F 2 "R1" H 4500 3950 60  0000 C CNN
+F 3 "" H 4800 3950 60  0000 C CNN
+	1    4800 3950
+	0    1    -1   0
+$EndComp
+$Comp
+L pulse v6
+U 1 1 5E283105
+P 7800 3800
+F 0 "v6" H 7600 3900 60  0000 C CNN
+F 1 "pulse" H 7600 3750 60  0000 C CNN
+F 2 "R1" H 7500 3800 60  0000 C CNN
+F 3 "" H 7800 3800 60  0000 C CNN
+	1    7800 3800
+	0    -1   1    0
+$EndComp
+Text Notes 9150 3450 0    60   ~ 0
+carry_in\n
+Text Notes 4550 2250 0    60   ~ 0
+A3
+Text Notes 4500 2800 0    60   ~ 0
+A4
+Text Notes 5050 4100 0    60   ~ 0
+a2
+Text Notes 7500 3750 0    60   ~ 0
+a1\n
 $EndSCHEMATC
