File: Examples/Analysis_Of_Digital_IC/4002_test/4002_test.sch (KiCad schematic (older format))
At the start: 32 parts, among them U1 adc_bridge_4, U10 plot_v1, U11 plot_v1, U12 plot_v1, U13 plot_v1, U2 dac_bridge_2, U3 adc_bridge_4, U4 plot_v1, U5 plot_v1, U6 plot_v1, U7 plot_v1, U8 plot_v1, U9 plot_v1, X1 IC_4002

Commit message: .pro files changed
Parts:
- v1, v2, v3, v4, v5, v6, v7, v8: symbol DC -> DC-RESCUE-4002_test
Changed lines of the file:
@@
 EESchema Schematic File Version 2
+LIBS:4002_test-rescue
 LIBS:power
+LIBS:eSim_Devices
+LIBS:eSim_User
+LIBS:eSim_Subckt
+LIBS:eSim_Sources
+LIBS:eSim_Power
+LIBS:eSim_Plot
+LIBS:eSim_Miscellaneous
+LIBS:eSim_Hybrid
+LIBS:eSim_Digital
 LIBS:eSim_Analog
-LIBS:eSim_Devices
-LIBS:eSim_Digital
-LIBS:eSim_Hybrid
-LIBS:eSim_Miscellaneous
-LIBS:eSim_Plot
-LIBS:eSim_Power
-LIBS:eSim_Sources
-LIBS:eSim_Subckt
-LIBS:eSim_User
+LIBS:4002_test-cache
 EELAYER 25 0
 EELAYER END
@@
 $EndComp
 $Comp
-L DC v6
+L DC-RESCUE-4002_test v6
 U 1 1 5CF1E4C8
 P 8200 3550
@@
 $EndComp
 $Comp
-L DC v5
+L DC-RESCUE-4002_test v5
 U 1 1 5CF1E4C2
 P 8200 3650
@@
 $EndComp
 $Comp
-L DC v8
+L DC-RESCUE-4002_test v8
 U 1 1 5CF1E4BC
 P 8200 3350
@@
 $EndComp
 $Comp
-L DC v7
+L DC-RESCUE-4002_test v7
 U 1 1 5CF1E4B6
 P 8200 3450
@@
 $EndComp
 $Comp
-L DC v4
+L DC-RESCUE-4002_test v4
 U 1 1 5CF1D11E
 P 2750 3550
@@
 $EndComp
 $Comp
-L DC v3
+L DC-RESCUE-4002_test v3
 U 1 1 5CF1D0EF
 P 2750 3450
@@
 $EndComp
 $Comp
-L DC v2
+L DC-RESCUE-4002_test v2
 U 1 1 5CF1D0C3
 P 2700 3350
@@
 $EndComp
 $Comp
-L DC v1
+L DC-RESCUE-4002_test v1
 U 1 1 5CF1CE2E
 P 2700 3250
