File: Examples/Analysis_Of_Digital_IC/4023_test/4023_test.sch (KiCad schematic (older format))
At the start: 26 parts, among them U1 plot_v1, U10 adc_bridge_3, U11 plot_v1, U12 plot_v1, U13 plot_v1, U14 plot_v1, U15 plot_v1, U16 plot_v1, U2 plot_v1, U3 plot_v1, U4 plot_v1, U5 plot_v1, U6 plot_v1, U7 adc_bridge_3, U8 adc_bridge_3, U9 dac_bridge_3, X1 4023

Commit message: .pro files changed
Parts:
- v1, v2, v3, v4, v5, v6, v7, v8, v9: symbol DC -> DC-RESCUE-4023_test
Changed lines of the file:
@@
 EESchema Schematic File Version 2
+LIBS:4023_test-rescue
 LIBS:power
 LIBS:eSim_Analog
@@
 LIBS:eSim_Plot
 LIBS:eSim_Power
-LIBS:eSim_PSpice
 LIBS:eSim_Sources
 LIBS:eSim_Subckt
 LIBS:eSim_User
+LIBS:4023_test-cache
 EELAYER 25 0
 EELAYER END
@@
 $EndComp
 $Comp
-L DC v1
+L DC-RESCUE-4023_test v1
 U 1 1 5CF24F1F
 P 1700 2350
@@
 $EndComp
 $Comp
-L DC v2
+L DC-RESCUE-4023_test v2
 U 1 1 5CF24F90
 P 1700 2900
@@
 $EndComp
 $Comp
-L DC v3
+L DC-RESCUE-4023_test v3
 U 1 1 5CF24FC7
 P 1700 3450
@@
 $EndComp
 $Comp
-L DC v4
+L DC-RESCUE-4023_test v4
 U 1 1 5CF25001
 P 1750 4000
@@
 $EndComp
 $Comp
-L DC v5
+L DC-RESCUE-4023_test v5
 U 1 1 5CF25044
 P 1750 4550
@@
 $EndComp
 $Comp
-L DC v6
+L DC-RESCUE-4023_test v6
 U 1 1 5CF25082
 P 1750 5050
@@
 	5950 5900 6200 5900
 $Comp
-L DC v7
+L DC-RESCUE-4023_test v7
 U 1 1 5CF25804
 P 9250 3250
@@
 $EndComp
 $Comp
-L DC v8
+L DC-RESCUE-4023_test v8
 U 1 1 5CF2580A
 P 9250 3800
@@
 $EndComp
 $Comp
-L DC v9
+L DC-RESCUE-4023_test v9
 U 1 1 5CF25810
 P 9250 4300
