File: Examples/Analysis_Of_Digital_IC/4028_test/4028_test.sch (KiCad schematic (older format))
At the start: 22 parts, among them U1 plot_v1, U10 plot_v1, U11 dac_bridge_8, U12 dac_bridge_2, U13 adc_bridge_4, U14 plot_v1, U15 plot_v1, U16 plot_v1, U17 plot_v1, U2 plot_v1, U3 plot_v1, U4 plot_v1, U5 plot_v1, U6 plot_v1, U7 plot_v1, U8 plot_v1, U9 plot_v1, X1 4028

Commit message: .pro files changed
Parts:
- v1, v2, v3, v4: symbol DC -> DC-RESCUE-4028_test
Changed lines of the file:
@@
 EESchema Schematic File Version 2
+LIBS:4028_test-rescue
 LIBS:power
 LIBS:eSim_Analog
@@
 LIBS:eSim_Subckt
 LIBS:eSim_User
+LIBS:4028_test-cache
 EELAYER 25 0
 EELAYER END
@@
 $EndComp
 $Comp
-L DC v2
+L DC-RESCUE-4028_test v2
 U 1 1 5CF25946
 P 9400 3950
@@
 $EndComp
 $Comp
-L DC v1
+L DC-RESCUE-4028_test v1
 U 1 1 5CF259A4
 P 9400 3400
@@
 $EndComp
 $Comp
-L DC v3
+L DC-RESCUE-4028_test v3
 U 1 1 5CF259F8
 P 9400 4500
@@
 $EndComp
 $Comp
-L DC v4
+L DC-RESCUE-4028_test v4
 U 1 1 5CF25A37
 P 9450 5000
