File: Examples/Analysis_Of_Digital_IC/4_Input_NAND_Charcateristics/4_Input_NAND_Charcateristics.sch (KiCad schematic (older format))
At the start: 22 parts, among them U1 plot_v1, U10 plot_v1, U11 plot_v1, U12 plot_v1, U13 plot_v1, U2 plot_v1, U3 plot_v1, U4 plot_v1, U5 adc_bridge_4, U6 plot_v1, U7 dac_bridge_2, U8 plot_v1, U9 adc_bridge_4, X1 4012

Commit message: .pro files changed
Parts:
- v1, v2, v3, v4, v5, v6, v7, v8: symbol DC -> DC-RESCUE-4_Input_NAND_Charcateristics
Changed lines of the file:
@@
 EESchema Schematic File Version 2
+LIBS:4_Input_NAND_Charcateristics-rescue
 LIBS:power
 LIBS:eSim_Analog
@@
 LIBS:eSim_Plot
 LIBS:eSim_Power
-LIBS:eSim_PSpice
 LIBS:eSim_Sources
 LIBS:eSim_User
@@
 NoConn ~ 5600 3750
 $Comp
-L DC v1
+L DC-RESCUE-4_Input_NAND_Charcateristics v1
 U 1 1 5CF2488C
 P 1900 3450
@@
 $EndComp
 $Comp
-L DC v2
+L DC-RESCUE-4_Input_NAND_Charcateristics v2
 U 1 1 5CF248E2
 P 1900 4000
@@
 $EndComp
 $Comp
-L DC v3
+L DC-RESCUE-4_Input_NAND_Charcateristics v3
 U 1 1 5CF24906
 P 1900 4550
@@
 $EndComp
 $Comp
-L DC v4
+L DC-RESCUE-4_Input_NAND_Charcateristics v4
 U 1 1 5CF24935
 P 1900 5100
@@
 $EndComp
 $Comp
-L DC v8
+L DC-RESCUE-4_Input_NAND_Charcateristics v8
 U 1 1 5CF24B50
 P 8150 4650
@@
 $EndComp
 $Comp
-L DC v7
+L DC-RESCUE-4_Input_NAND_Charcateristics v7
 U 1 1 5CF24B56
 P 8150 4100
@@
 $EndComp
 $Comp
-L DC v6
+L DC-RESCUE-4_Input_NAND_Charcateristics v6
 U 1 1 5CF24B5C
 P 8150 3550
@@
 $EndComp
 $Comp
-L DC v5
+L DC-RESCUE-4_Input_NAND_Charcateristics v5
 U 1 1 5CF24B62
 P 8150 3000
